Commit message: caster wheels added

File: urdf/barista_robot_model.urdf (robot description, URDF)
Before this commit: robot barista_robot, 9 links, 8 joints
Links:
- added link back_pitch_link; visual sphere radius=0.0242
- added link back_roll_link; visual cylinder length=0.002 radius=0.005
- added link back_yaw_link; visual cylinder length=0.002 radious=0.005
- added link front_pitch_link; visual sphere radius=0.0242
- added link front_roll_link; visual cylinder length=0.002 radius=0.005
- added link front_yaw_link; visual cylinder length=0.002 radious=0.005
Joints:
- added joint back_pitch_joint: type continuous, parent back_roll_link, child back_pitch_link, origin xyz=0 0 0 rpy=0 0 0, axis 0 1 0
- added joint back_roll_joint: type continuous, parent back_yaw_link, child back_roll_link, origin xyz=0 0 0 rpy=0 0 0, axis 1 0 0
- added joint back_yaw_joint: type continuous, parent base_body, child back_yaw_link, origin xyz=-0.120 0 -0.0753 rpy=0 0 0, axis 0 0 1
- added joint front_pitch_joint: type continuous, parent front_roll_link, child front_pitch_link, origin xyz=0 0 0 rpy=0 0 0, axis 0 1 0
- added joint front_roll_joint: type continuous, parent front_yaw_link, child front_roll_link, origin xyz=0 0 0 rpy=0 0 0, axis 1 0 0
- added joint front_yaw_joint: type continuous, parent base_body, child front_yaw_link, origin xyz=0.120 0 -0.0753 rpy=0 0 0, axis 0 0 1
- joint base_link_joint: origin xyz=0 0 0.0951 rpy=0 0 0 -> xyz=0 0 0.0995 rpy=0 0 0
- joint joint_wheel_left: origin xyz=0.0 0.150 -0.0775 rpy=0 0 0 -> xyz=0.0 0.150 -0.0643 rpy=0 0 0
- joint joint_wheel_right: origin xyz=0.0 -0.150 -0.0775 rpy=0 0 0 -> xyz=0.0 -0.150 -0.0643 rpy=0 0 0

Commit message: laser added

File: urdf/barista_robot_model.urdf (robot description, URDF)
Before this commit: robot barista_robot, 15 links, 14 joints
Links:
- added link laser_scan_link; visual mesh filename=package://barista_robot_description/meshes/slamtec_rplidar_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 scale=1 1 1
- link back_yaw_link: geometry visual cylinder length=0.002 radius=0.005
- link front_yaw_link: geometry visual cylinder length=0.002 radius=0.005
Joints:
- added joint laser_scan_link_joint: type prismatic, parent base_body, child laser_scan_link, origin xyz=0.110 0 0.0775 rpy=0 0 0, limit lower=-0.1 upper=0.0 effort=20.0 velocity=2.0

Commit message: all plugins added, gazebo test ok, topic: laser, odom ok

File: urdf/barista_robot_model.urdf (robot description, URDF)
Before this commit: robot barista_robot, 16 links, 15 joints
Links:
- added link laser_scan_frame
- added link laser_scan_model_link, mass 0.01; collision cylinder length=0.0408 radius=0.037493; visual mesh filename=package://barista_robot_description/meshes/slamtec_rplidar_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 scale=1.0 1.0 1.0
- link back_pitch_link: mass None -> 0.05; geometry collision sphere radius=0.0242; visual sphere radius=0.0242
- link back_roll_link: mass None -> 0.01; geometry collision cylinder length=0.002 radius=0.005; visual cylinder length=0.002 radius=0.005
- link back_yaw_link: mass None -> 0.01; geometry collision cylinder length=0.002 radius=0.005; visual cylinder length=0.002 radius=0.005
- link base_body: mass None -> 7.0; geometry collision cylinder length=0.155 radius=0.178; visual cylinder length=0.155 radius=0.178
- link base_head: mass None -> 2.0; geometry collision cylinder length=0.090 radius=0.160; visual cylinder length=0.090 radius=0.160
- link base_standoff_left_negative: mass None -> 0.18; geometry collision cylinder length=0.220 radius=0.010; visual cylinder length=0.220 radius=0.010
- link base_standoff_left_positive: mass None -> 0.18; geometry collision cylinder length=0.220 radius=0.010; visual cylinder length=0.220 radius=0.010
- link base_standoff_right_negative: mass None -> 0.18; geometry collision cylinder length=0.220 radius=0.010; visual cylinder length=0.220 radius=0.010
- link base_standoff_right_positive: mass None -> 0.18; geometry collision cylinder length=0.220 radius=0.010; visual cylinder length=0.220 radius=0.010
- link base_wheel_left: mass None -> 0.5; geometry collision cylinder length=0.0206 radius=0.0352; visual cylinder length=0.0206 radius=0.0352
- link base_wheel_right: mass None -> 0.5; geometry collision cylinder length=0.0206 radius=0.0352; visual cylinder length=0.0206 radius=0.0352
- link front_pitch_link: mass None -> 0.05; geometry collision sphere radius=0.0242; visual sphere radius=0.0242
- link front_roll_link: mass None -> 0.01; geometry collision cylinder length=0.002 radius=0.005; visual cylinder length=0.002 radius=0.005
- link front_yaw_link: mass None -> 0.01; geometry collision cylinder length=0.002 radius=0.005; visual cylinder length=0.002 radius=0.005
- link laser_scan_link: mass None -> 0.01; geometry collision box size=0.02 0.02 0.02; visual box size=0.02 0.02 0.02
Joints:
- added joint laser_scan_frame_joint: type fixed, parent laser_scan_link, child laser_scan_frame, origin xyz=0 0 0.0408 rpy=0 0 0
- added joint laser_scan_model_link_joint: type continuous, parent laser_scan_link, child laser_scan_model_link, origin xyz=0.0 0.0 0.0 rpy=0 0 0, axis 0 0 1, limit effort=10.0 velocity=2.0
- joint back_pitch_joint: limit (none) -> effort=1000.0 velocity=100.0
- joint back_roll_joint: limit (none) -> effort=1000.0 velocity=100.0
- joint back_yaw_joint: limit (none) -> effort=1000.0 velocity=100.0
- joint front_pitch_joint: limit (none) -> effort=1000.0 velocity=100.0
- joint front_roll_joint: limit (none) -> effort=1000.0 velocity=100.0
- joint front_yaw_joint: limit (none) -> effort=1000.0 velocity=100.0
- joint joint_wheel_left: limit (none) -> effort=10000 velocity=1000
- joint joint_wheel_right: limit (none) -> effort=10000 velocity=1000
- joint laser_scan_link_joint: axis (none) -> 0 0 1; origin xyz=0.110 0 0.0775 rpy=0 0 0 -> xyz=0.110 0.0 0.0775 rpy=0 0 0
