Commit message: launch file modified to include laser or not, changes in xacro to use laser and ros2_control with plugins

File: xacro/barista_robot_model.urdf.xacro (robot description, xacro)
@@ -1,4 +1,14 @@
 <?xml version="1.0"?>
 <robot xmlns:xacro="http://www.ros.org/wiki/xacro" name="barista_robot">
+<!-- ____________________________ Materials defined for this robot____________-->
+<material name="blue">
+<color rgba="0.0 0.0 1.0 1"/>
+</material>
+<material name="gray">
+<color rgba="0.5 0.5 0.5 1"/>
+</material>
+<material name="rubber_black">
+<color rgba="0.05 0.05 0.05 1"/>
+</material>
 <!-- include gazebo tags-->
 <xacro:include filename="$(find barista_robot_description)/xacro/drive_wheel.xacro"/>
@@ -6,4 +16,5 @@
 <xacro:include filename="$(find barista_robot_description)/xacro/standoff_rod.xacro"/>
 <xacro:include filename="$(find barista_robot_description)/xacro/cup_holder_tray.xacro"/>
+<xacro:include filename="$(find barista_robot_description)/xacro/laser_scanner.xacro"/>
 <!-- main properties for the robot-->
 <xacro:property name="body_radius" value="0.178"/>
@@ -16,5 +27,5 @@
 <xacro:property name="cup_tray_radius" value="0.160"/>
 <xacro:property name="cup_tray_length" value="0.090"/>
-<xacro:arg name="include_laser" default="true"/>
+<xacro:arg name="include_laser" default="false"/>
 <!-- ____________________________ Base link______________________________________ -->
 <link name="base_link">
@@ -58,100 +69,9 @@
 <!--___________________________Including the cup tray (based_head)___________-->
 <xacro:cup_holder_tray radius="${cup_tray_radius}" length="${cup_tray_length}"/>
-<!--___________________________Defining xacro macro__________________________-->
-<!--Laser scan-->
-<!-- Laser Position Control -->
-<xacro:macro name="Laser_scanner">
-  <link name="laser_scan_link">
-    <visual>
-      <origin rpy="0 0 0" xyz="0 0 0"/>
-      <geometry>
-        <box size="0.02 0.02 0.02"/>
-      </geometry>
-    </visual>
-    <collision>
-       <origin rpy="0 0 0" xyz="0 0 0.0204"/>
-      <geometry>
-        <box size="0.02 0.02 0.02"/>
-      </geometry>
-    </collision>
-    <inertial>
-      <mass value="0.01"/>
-      <origin rpy="0 0 0" xyz="0 0 0.0204"/>
-      <inertia ixx="6.066578520833334e-06" ixy="0" ixz="0" iyy="6.072950163333333e-06" iyz="0" izz="9.365128684166666e-06"/>
-    </inertial>
-  </link>
-  <joint name="laser_scan_link_joint" type="prismatic">
-    <origin rpy="0 0 0" xyz="0.110 0.0 0.0775"/>
-    <parent link="base_body"/>
-    <child link="laser_scan_link"/>
-    <axis xyz="0 0 1"/>
-    <limit lower="-0.1" upper="0.0" effort="20.0" velocity="2.0"/>
-    <dynamics damping="0.1" friction="1.0"/>
-  </joint>
-  <link name="laser_scan_frame">
-  </link>
-  <joint name="laser_scan_frame_joint" type="fixed">
-    <origin rpy="0 0 0" xyz="0 0 0.0408"/>
-    <parent link="laser_scan_link"/>
-    <child link="laser_scan_frame"/>
-  </joint>
-  <!-- Visual Laser Model to be rotated -->
-  <link name="laser_scan_model_link">
-    <visual>
-      <origin rpy="0 0 0" xyz="0 0 0"/>
-      <geometry>
-        <mesh filename="package://barista_robot_description/meshes/slamtec_rplidar_a2m8.dae" scale="1.0 1.0 1.0"/>
-      </geometry>
-    </visual>
-    <collision>
-       <origin rpy="0 0 0" xyz="0 0 0.0204"/>
-      <geometry>
-        <cylinder length="0.0408" radius="0.037493"/>
-      </geometry>
-    </collision>
-    <inertial>
-      <mass value="0.01"/>
-      <origin rpy="0 0 0" xyz="0 0 0.0204"/>
-      <inertia ixx="6.066578520833334e-06" ixy="0" ixz="0" iyy="6.072950163333333e-06" iyz="0" izz="9.365128684166666e-06"/>
-    </inertial>
-  </link>
-  <joint name="laser_scan_model_link_joint" type="continuous">
-    <origin rpy="0 0 0" xyz="0.0 0.0 0.0"/>
-    <parent link="laser_scan_link"/>
-    <child link="laser_scan_model_link"/>
-    <axis xyz="0 0 1"/>
-    <limit effort="10.0" velocity="2.0"/>
-    <dynamics friction="0.01"/>
-  </joint>
-<!-- Laser Scanner Plugin -->
-<gazebo reference="laser_scan_frame">
-<sensor type="gpu_lidar" name="gpu_lidar">
-<pose relative_to='laser_scan_frame'>0 0 0 0 0 0</pose>
-<gz_frame_id>laser_scan_frame</gz_frame_id>
-<always_on>1</always_on>
-<visualize>true</visualize>
-<update_rate>100</update_rate>
-<topic>/laser_scan</topic>
-<ray>
-<scan>
-<horizontal>
-<samples>200</samples>
-<resolution>1</resolution>
-<min_angle>-3.14</min_angle>
-<max_angle>3.14</max_angle>
-</horizontal>
-</scan>
-<range>
-<min>0.1</min>
-<max>5.0</max>
-<resolution>0.01</resolution>
-</range>
-</ray>
-</sensor>
-</gazebo>
-</xacro:macro>
 <!--___________________________Including Laser with conditional_________________________-->
 <xacro:if value="$(arg include_laser)">
     <xacro:Laser_scanner/>
+</xacro:if>
+<xacro:if value="$(arg include_laser)">
     <!-- ros2_control config -->
     <ros2_control name="GazeboSimSystem" type="system">
@@ -179,4 +99,12 @@
     </joint>
     </ros2_control>
+    <!-- Gazebo Sim system plugin that boots the controller manager and parses the ros2_control tags -->
+    <gazebo>
+    <plugin filename="gz_ros2_control-system"
+    name="gz_ros2_control::GazeboSimROS2ControlPlugin">
+    <!-- Controller configuration YAML file -->
+    <parameters>$(find barista_robot_description)/config/controller_position_velocity.yaml</parameters>
+    </plugin>
+    </gazebo>
 </xacro:if>
 <!-- ______________________________PLUGINS for the robot, velocity, laser, etc-->
@@ -223,12 +151,4 @@
 </plugin>
 </gazebo>
-<!-- Gazebo Sim system plugin that boots the controller manager and parses the ros2_control tags -->
-<gazebo>
-<plugin filename="gz_ros2_control-system"
-name="gz_ros2_control::GazeboSimROS2ControlPlugin">
-<!-- Controller configuration YAML file -->
-<parameters>$(find barista_robot_description)/config/controller_position_velocity.yaml</parameters>
-</plugin>
-</gazebo>
 <!-- ___________________________________________________ Enable Sensors in Gazebo Sim -->
 <gazebo>
